File: boards/eater-6502-sbc/eater-6502-sbc.kicad_sch (KiCad schematic)
At the start: 43 parts, among them J1 Jack-DC, J2 JMP_CLK, J3 EXT_CLK, SW1 SW_RST, U1 LM317_TO-220, U2 W65C02S, U3 28C256, U4 KM62256CLP, U5 W65C22S, U6 74HC00

Commit message: SBC design 2 start
Parts:
- removed C? (x6): 1u, symbol Device:C_Small
- C1: footprint (none) -> Capacitor_THT:C_Disc_D3.4mm_W2.1mm_P2.50mm
- C11, C13, C15, C4, C5, C7, C9: renamed from C?; footprint (none) -> C_Disc_D3.4mm_W2.1mm_P2.50mm
- C2: footprint (none) -> Capacitor_THT:CP_Radial_D4.0mm_P1.50mm
- C3: footprint (none) -> Capacitor_THT:CP_Radial_D5.0mm_P2.00mm
- D3: footprint (none) -> Diode_THT:D_DO-41_SOD81_P7.62mm_Horizontal
- D4: renamed from D?; value LED -> PWR_LED; footprint (none) -> LED_THT:LED_D5.0mm
- F1: footprint (none) -> Fuse:Fuse_BelFuse_0ZRE0005FF_L8.3mm_W3.8mm
- R1, R2: footprint (none) -> Resistor_THT:R_Axial_DIN0207_L6.3mm_D2.5mm_P10.16mm_Horizontal
- R3, R5, R6, R7: renamed from R?; footprint (none) -> Resistor_THT:R_Axial_DIN0204_L3.6mm_D1.6mm_P5.08mm_Horizontal
- R4: renamed from R?; value R -> 1k; footprint (none) -> Resistor_THT:R_Axial_DIN0204_L3.6mm_D1.6mm_P5.08mm_Horizontal
- SW1: footprint (none) -> Button_Switch_THT:SW_PUSH_6mm
- U6: footprint Package_DIP:DIP-8_W7.62mm_LongPads -> Package_DIP:DIP-14_W7.62mm_LongPads
- gave numbers to parts that had none: 3
