File: boards/eater-6502-sbc-2/eater-6502-sbc-2.kicad_pcb (KiCad board)
At the start: 2 copper layers, 89 x 112 mm, 37 parts, among them J1 HDR_EXT_CLK, J2 HDR_CPU_BUS, J3 Jack-DC, J4 HDR_PA[0:4], SW1 SW_RESET, SW2 SW_SPDT, U1 W65C02SxP, U2 28C256, U3 KM62256CLP, U4 W65C22NxP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

Commit message: Finished rough layout and parts selection.
Parts:
- removed DS1: WC1602A, Display:WC1602A
- removed RV1: 10k, Potentiometer_THT:Potentiometer_Piher_PT-6-V_Vertical_Hole
- added H1: M3, MountingHole:MountingHole_3.2mm_M3_Pad, F.Cu at (141.5, 31.8)
- added H2: M3, MountingHole:MountingHole_3.2mm_M3_Pad, F.Cu at (230.4, 31.8)
- added H3: M3, MountingHole:MountingHole_3.2mm_M3_Pad, F.Cu at (230.4, 120.7)
- added H4: M3, MountingHole:MountingHole_3.2mm_M3_Pad, F.Cu at (141.5, 120.7)
- C1, C3, C5, C7, C9: footprint Capacitor_THT:C_Rect_L4.6mm_W5.5mm_P2.50mm_MKS02_FKP02 -> Capacitor_THT:C_Rect_L4.0mm_W2.5mm_P2.50mm
- C12: footprint Capacitor_THT:C_Rect_L4.6mm_W5.5mm_P2.50mm_MKS02_FKP02 -> Capacitor_THT:CP_Radial_D4.0mm_P1.50mm
- J4: value HDR_PA[0:4] -> HDR_PIO_PORT; footprint Connector_PinSocket_2.54mm:PinSocket_1x05_P2.54mm_Vertical -> Connector_PinSocket_2.54mm:PinSocket_1x20_P2.54mm_Vertical
- SW2: value SW_SPDT -> SW_PWR; footprint Button_Switch_THT:SW_Slide_1P2T_CK_OS102011MS2Q -> EaterLibrary:Button_Switch_SPST_NKK_CS12ANW03
- U2: footprint Socket:DIP_Socket-28_W11.9_W12.7_W15.24_W17.78_W18.5_3M_228-1277-00-0602J -> Package_DIP:DIP-28_W15.24mm_Socket_LongPads
- U3: footprint Package_DIP:DIP-28_W15.24mm -> Package_DIP:DIP-28_W15.24mm_Socket_LongPads
- U5: value 74HC00 -> 74HC132
- U6: value LM7805_TO220 -> MC7805
- moved J4 197.0 mm to (231.6, 52.1)
- moved J1 161.3 mm to (225.5, 44.7), turned to 180 degrees
- moved U5 158.8 mm to (217.2, 106.7)
- moved C10 144.3 mm to (228.6, 106.7)
- moved R4 140.5 mm to (196.8, 62.2), turned to 90 degrees
- moved R1 127.5 mm to (167.6, 48.0)
- moved C9 126.3 mm to (229.9, 110.5), turned to -90 degrees
- moved U6 124.0 mm to (153.4, 47.0), turned to -90 degrees
- moved JP1 122.0 mm to (207.0, 39.4)
- moved SW1 116.6 mm to (184.4, 47.7), turned to 90 degrees
- moved C8 114.0 mm to (199.4, 100.3), turned to 180 degrees
- moved R5 112.5 mm to (196.1, 47.0), turned to -90 degrees
- moved R2 112.4 mm to (175.3, 48.0)
- moved C11 108.8 mm to (193.0, 45.7), turned to -90 degrees
- moved SW2 108.5 mm to (140.5, 47.4)
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Connections:
- HS1 pad 1: (no net) -> unconnected-(HS1-Pad1)
- U4 pad 18: unconnected-(U4-Pad18) -> /CB1
- U4 pad 19: unconnected-(U4-Pad19) -> /CB2
- U4 pad 39: unconnected-(U4-Pad39) -> /CA2
- U4 pad 40: unconnected-(U4-Pad40) -> /CA1
Other:
- board size 89 x 112 mm -> 99.1 x 99.1 mm
- board text added: "18V DC Max"
- board text added: "AT28C256"
- board text added: "CLK In"
- board text added: "CXO"
- board text added: "Eater 6502 - Memory Map RAM: 0x0000 - 0x3FFF IO: 0x4000 - 0x7FFF ROM: 0x8000 - 0xFFFF"
- board text added: "External Clock"
- board text added: "Ground"
- board text added: "OFF"
- board text added: "ON"
- board text added: "PWR"
- board text added: "Reset"
- board text added: "~{RST}"
